File: PowerLatch.brd (EAGLE design)
At the start: 8.9 x 9.4 mm, 10 parts, among them J1 455-1750-1-ND, J2 455-1750-1-ND, Q1 FDC365P, Q2 BFN26

Commit message: Rev. 1.0
Parts:
- added LOGO1: OSHW-LOGOS, SparkFun-Aesthetics:OSHW-LOGO-S
Other:
- board size 8.9 x 9.4 mm -> 9.4 x 9.4 mm
- board text added: "PowerLatch rev. 1.0 psyte - 2019"
Changed lines of the file:
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@@
 <?xml version="1.0" encoding="utf-8"?>
 <!DOCTYPE eagle SYSTEM "eagle.dtd">
-<eagle version="9.1.3">
+<eagle version="9.4.0">
 <drawing>
 <settings>
@@
 <fusionsync huburn="a.cGVyc29uYWw6dWUyZDY1NDI2" projecturn="a.cGVyc29uYWw6dWUyZDY1NDI2IzIwMTgwOTMwMTUxNzkxMzAx" f3durn="urn:adsk.wipprod:dm.lineage:l-7Gt0VZT-20rkTW2Obkdw" pcbguid="1a52890b-5eb1-4531-954d-5ca6c4217f20" lastpulledtime="" lastsyncedchangeguid="5de202c5-14e5-fb1e-5878-0e9cb41dfa64"/>
 <plain>
-<wire x1="5.08" y1="1.651" x2="13.97" y2="1.651" width="0" layer="20"/>
-<wire x1="13.97" y1="1.651" x2="13.97" y2="11.049" width="0" layer="20"/>
-<wire x1="13.97" y1="11.049" x2="5.08" y2="11.049" width="0" layer="20"/>
-<wire x1="5.08" y1="11.049" x2="5.08" y2="1.651" width="0" layer="20"/>
-<dimension x1="5.08" y1="1.27" x2="13.97" y2="1.27" x3="9.525" y3="-1.27" textsize="1.778" layer="47"/>
+<wire x1="4.826" y1="1.651" x2="14.224" y2="1.651" width="0" layer="20"/>
+<wire x1="14.224" y1="1.651" x2="14.224" y2="11.049" width="0" layer="20"/>
+<wire x1="14.224" y1="11.049" x2="4.826" y2="11.049" width="0" layer="20"/>
+<wire x1="4.826" y1="11.049" x2="4.826" y2="1.651" width="0" layer="20"/>
+<dimension x1="4.826" y1="1.27" x2="14.224" y2="1.27" x3="9.525" y3="-1.27" textsize="1.778" layer="47"/>
 <dimension x1="13.97" y1="1.651" x2="13.97" y2="11.049" x3="17.78" y3="6.35" textsize="1.778" layer="47"/>
 <wire x1="7.62" y1="9.906" x2="7.62" y2="9.144" width="0.254" layer="21"/>
 <wire x1="7.239" y1="8.509" x2="7.239" y2="7.747" width="0.254" layer="21"/>
+<text x="9.271" y="2.286" size="0.8128" layer="22" font="vector" ratio="20" rot="MR90">PowerLatch
+rev. 1.0
+psyte - 2019</text>
 </plain>
 <attributes>
@@
 <attribute name="SPICEPREFIX" value="R" x="7.874" y="5.08" size="1.778" layer="27" display="off"/>
 </element>
+<element name="LOGO1" library="SparkFun-Aesthetics" package="OSHW-LOGO-S" value="OSHW-LOGOS" x="7.62" y="6.35" smashed="yes" rot="MR90"/>
 </elements>
 <signals>
@@
 </drawing>
 <compatibility>
+<note version="6.3" minversion="6.2.2" severity="warning">
+Since Version 6.2.2 text objects can contain more than one line,
+which will not be processed correctly with this version.
+</note>
 <note version="8.2" severity="warning">
 Since Version 8.2, EAGLE supports online libraries. The ids
