File: PowerLatch.sch (EAGLE design)
At the start: 10 parts, among them J1 455-1750-1-ND, J2 455-1750-1-ND, Q1 FDC365P, Q2 BFN26

Commit message: Rev. 1.0
Parts:
- added LOGO1: OSHW-LOGOS, SparkFun-Aesthetics:OSHW-LOGOS
Changed lines of the file:
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@@
 <?xml version="1.0" encoding="utf-8"?>
 <!DOCTYPE eagle SYSTEM "eagle.dtd">
-<eagle version="9.1.3">
+<eagle version="9.4.0">
 <drawing>
 <settings>
@@
 <part name="P+4" library="supply1" library_urn="urn:adsk.eagle:library:371" deviceset="+5V" device="" value="VCC"/>
 <part name="GND3" library="supply1" library_urn="urn:adsk.eagle:library:371" deviceset="GND" device=""/>
+<part name="LOGO1" library="SparkFun-Aesthetics" deviceset="OSHW-LOGO" device="S"/>
 </parts>
 <sheets>
@@
 </plain>
 <instances>
-<instance part="Q1" gate="G$1" x="22.86" y="93.98" rot="MR90"/>
-<instance part="Q2" gate="G$1" x="30.48" y="73.66" rot="MR0"/>
-<instance part="R1" gate="G$1" x="10.16" y="88.9" rot="R90"/>
-<instance part="C1" gate="G$1" x="10.16" y="73.66"/>
-<instance part="R2" gate="G$1" x="40.64" y="73.66" rot="R180"/>
-<instance part="GND1" gate="1" x="27.94" y="48.26"/>
-<instance part="P+1" gate="1" x="5.08" y="111.76" rot="MR0"/>
-<instance part="P+2" gate="1" x="40.64" y="111.76"/>
-<instance part="GND2" gate="1" x="91.44" y="83.82"/>
-<instance part="R3" gate="G$1" x="48.26" y="66.04" rot="R270"/>
+<instance part="Q1" gate="G$1" x="22.86" y="93.98" smashed="yes" rot="MR90">
+<attribute name="NAME" x="22.86" y="99.06" size="1.778" layer="95" font="vector" rot="MR90"/>
+<attribute name="VALUE" x="20.32" y="99.06" size="1.778" layer="96" font="vector" rot="MR90"/>
+</instance>
+<instance part="Q2" gate="G$1" x="30.48" y="73.66" smashed="yes" rot="MR0">
+<attribute name="NAME" x="27.94" y="73.66" size="1.778" layer="95" font="vector" rot="MR0"/>
+<attribute name="VALUE" x="27.94" y="71.374" size="1.778" layer="96" font="vector" rot="MR0"/>
+</instance>
+<instance part="R1" gate="G$1" x="10.16" y="88.9" smashed="yes" rot="R90">
+<attribute name="NAME" x="8.6614" y="85.09" size="1.778" layer="95" rot="R90"/>
+<attribute name="VALUE" x="13.462" y="85.09" size="1.778" layer="96" rot="R90"/>
+</instance>
+<instance part="C1" gate="G$1" x="10.16" y="73.66" smashed="yes">
+<attribute name="NAME" x="11.684" y="74.041" size="1.778" layer="95"/>
+<attribute name="VALUE" x="11.684" y="68.961" size="1.778" layer="96"/>
+</instance>
+<instance part="R2" gate="G$1" x="40.64" y="73.66" smashed="yes" rot="R180">
+<attribute name="NAME" x="44.45" y="72.1614" size="1.778" layer="95" rot="R180"/>
+<attribute name="VALUE" x="44.45" y="76.962" size="1.778" layer="96" rot="R180"/>
+</instance>
+<instance part="GND1" gate="1" x="27.94" y="48.26" smashed="yes">
+<attribute name="VALUE" x="25.4" y="45.72" size="1.778" layer="96"/>
+</instance>
+<instance part="P+1" gate="1" x="5.08" y="111.76" smashed="yes" rot="MR0">
+<attribute name="VALUE" x="7.62" y="106.68" size="1.778" layer="96" rot="MR90"/>
+</instance>
+<instance part="P+2" gate="1" x="40.64" y="111.76" smashed="yes">
+<attribute name="VALUE" x="38.1" y="106.68" size="1.778" layer="96" rot="R90"/>
+</instance>
+<instance part="GND2" gate="1" x="91.44" y="83.82" smashed="yes">
+<attribute name="VALUE" x="88.9" y="81.28" size="1.778" layer="96"/>
+</instance>
+<instance part="R3" gate="G$1" x="48.26" y="66.04" smashed="yes" rot="R270">
+<attribute name="NAME" x="49.7586" y="69.85" size="1.778" layer="95" rot="R270"/>
+<attribute name="VALUE" x="44.958" y="69.85" size="1.778" layer="96" rot="R270"/>
+</instance>
 <instance part="J1" gate="J$1" x="-30.48" y="91.44" smashed="yes">
 <attribute name="NAME" x="-33.02" y="97.028" size="1.778" layer="95" font="vector"/>
@@
 <attribute name="VALUE" x="-22.86" y="81.788" size="1.778" layer="96"/>
 </instance>
-<instance part="GND3" gate="1" x="-20.32" y="66.04"/>
+<instance part="GND3" gate="1" x="-20.32" y="66.04" smashed="yes">
+<attribute name="VALUE" x="-22.86" y="63.5" size="1.778" layer="96"/>
+</instance>
+<instance part="LOGO1" gate="G$1" x="73.66" y="50.8" smashed="yes"/>
 </instances>
 <busses>
